Commit message: fix: remove fixed wheelchair caster ground contact

File: urdf/wheelchair.xacro (robot description, xacro)
@@ -69,11 +69,12 @@
   <xacro:wheel name="left_wheel" y="${sep/2}"/>
   <xacro:wheel name="right_wheel" y="${-sep/2}"/>
-  <!-- passive front caster (sphere) -->
+  <!-- Passive front caster visual. This link is fixed to the chassis and has
+       no steer/roll degree of freedom; a ground collision here creates a
+       third, non-holonomic contact that physically locks diff-drive yaw.
+       The two driven wheels are the only ground-contact geometry. -->
   <link name="caster">
     <inertial><mass value="0.5"/>
       <inertia ixx="0.001" ixy="0" ixz="0" iyy="0.001" iyz="0" izz="0.001"/></inertial>
     <visual><geometry><sphere radius="0.06"/></geometry><material name="dark"/></visual>
-    <collision><geometry><sphere radius="0.06"/></geometry>
-      <surface><friction><ode><mu>0.0</mu><mu2>0.0</mu2></ode></friction></surface></collision>
   </link>
   <joint name="caster_joint" type="fixed">
@@ -82,5 +83,4 @@
     <origin xyz="${base_x/2 - 0.1} 0 ${-base_z/2 - wheel_r + 0.06}"/>
   </joint>
-  <gazebo reference="caster"><mu1>0.0</mu1><mu2>0.0</mu2></gazebo>
   <gazebo reference="left_wheel"><mu1>1.0</mu1><mu2>1.0</mu2></gazebo>
   <gazebo reference="right_wheel"><mu1>1.0</mu1><mu2>1.0</mu2></gazebo>

Commit message: revert: retain wheelchair caster collision

File: urdf/wheelchair.xacro (robot description, xacro)
@@ -69,12 +69,11 @@
   <xacro:wheel name="left_wheel" y="${sep/2}"/>
   <xacro:wheel name="right_wheel" y="${-sep/2}"/>
-  <!-- Passive front caster visual. This link is fixed to the chassis and has
-       no steer/roll degree of freedom; a ground collision here creates a
-       third, non-holonomic contact that physically locks diff-drive yaw.
-       The two driven wheels are the only ground-contact geometry. -->
+  <!-- passive front caster (sphere) -->
   <link name="caster">
     <inertial><mass value="0.5"/>
       <inertia ixx="0.001" ixy="0" ixz="0" iyy="0.001" iyz="0" izz="0.001"/></inertial>
     <visual><geometry><sphere radius="0.06"/></geometry><material name="dark"/></visual>
+    <collision><geometry><sphere radius="0.06"/></geometry>
+      <surface><friction><ode><mu>0.0</mu><mu2>0.0</mu2></ode></friction></surface></collision>
   </link>
   <joint name="caster_joint" type="fixed">
@@ -83,4 +82,5 @@
     <origin xyz="${base_x/2 - 0.1} 0 ${-base_z/2 - wheel_r + 0.06}"/>
   </joint>
+  <gazebo reference="caster"><mu1>0.0</mu1><mu2>0.0</mu2></gazebo>
   <gazebo reference="left_wheel"><mu1>1.0</mu1><mu2>1.0</mu2></gazebo>
   <gazebo reference="right_wheel"><mu1>1.0</mu1><mu2>1.0</mu2></gazebo>

Commit message: test: audit wheelchair contact physics

File: urdf/wheelchair.xacro (robot description, xacro)
@@ -7,4 +7,5 @@
   <xacro:property name="wheel_w" value="0.05"/>
   <xacro:property name="sep" value="0.62"/>
+  <xacro:arg name="wheel_mu" default="1.0"/>
   <material name="chair"><color rgba="0.2 0.3 0.4 1"/></material>
   <material name="dark"><color rgba="0.1 0.1 0.1 1"/></material>
@@ -83,6 +84,26 @@
   </joint>
   <gazebo reference="caster"><mu1>0.0</mu1><mu2>0.0</mu2></gazebo>
-  <gazebo reference="left_wheel"><mu1>1.0</mu1><mu2>1.0</mu2></gazebo>
-  <gazebo reference="right_wheel"><mu1>1.0</mu1><mu2>1.0</mu2></gazebo>
+  <gazebo reference="left_wheel">
+    <mu1>$(arg wheel_mu)</mu1><mu2>$(arg wheel_mu)</mu2>
+    <sensor name="left_wheel_contact_sensor" type="contact">
+      <always_on>true</always_on><update_rate>100</update_rate>
+      <contact><collision>left_wheel_collision</collision></contact>
+      <plugin name="left_wheel_contact_plugin" filename="libgazebo_ros_bumper.so">
+        <bumperTopicName>/wheelchair/left_wheel/contact</bumperTopicName>
+        <frameName>left_wheel</frameName>
+      </plugin>
+    </sensor>
+  </gazebo>
+  <gazebo reference="right_wheel">
+    <mu1>$(arg wheel_mu)</mu1><mu2>$(arg wheel_mu)</mu2>
+    <sensor name="right_wheel_contact_sensor" type="contact">
+      <always_on>true</always_on><update_rate>100</update_rate>
+      <contact><collision>right_wheel_collision</collision></contact>
+      <plugin name="right_wheel_contact_plugin" filename="libgazebo_ros_bumper.so">
+        <bumperTopicName>/wheelchair/right_wheel/contact</bumperTopicName>
+        <frameName>right_wheel</frameName>
+      </plugin>
+    </sensor>
+  </gazebo>
   <gazebo>
     <plugin name="gazebo_ros_control" filename="libgazebo_ros_control.so">

Commit message: test: parameterize wheelchair drive authority

File: urdf/wheelchair.xacro (robot description, xacro)
@@ -8,4 +8,8 @@
   <xacro:property name="sep" value="0.62"/>
   <xacro:arg name="wheel_mu" default="1.0"/>
+  <!-- Explicit, symmetric velocity-loop authority.  The probe may vary only
+       effort; velocity remains bounded above the 1.333 rad/s test target. -->
+  <xacro:arg name="wheel_effort_limit" default="10.0"/>
+  <xacro:arg name="wheel_velocity_limit" default="4.0"/>
   <!-- Disabled by default: the probe can enable an explicit ODE friction
        direction without changing the production isotropic-contact baseline. -->
@@ -77,4 +81,5 @@
       <origin xyz="0 ${y} ${-base_z/2}"/>
       <axis xyz="0 1 0"/>
+      <limit effort="$(arg wheel_effort_limit)" velocity="$(arg wheel_velocity_limit)"/>
     </joint>
     <transmission name="${name}_trans">

Commit message: fix: simplify wheelchair diff drive chassis

File: urdf/wheelchair.xacro (robot description, xacro)
@@ -33,6 +33,8 @@
   <link name="base_link">
     <inertial>
-      <mass value="40"/>
-      <inertia ixx="2.0" ixy="0" ixz="0" iyy="2.0" iyz="0" izz="2.0"/>
+      <!-- Minimal standard diff-drive execution body.  Dimensions remain the
+           wheelchair footprint; only its physical carrier is simplified. -->
+      <mass value="12.0"/>
+      <inertia ixx="0.45" ixy="0" ixz="0" iyy="0.56" iyz="0" izz="0.73"/>
     </inertial>
     <visual>
@@ -55,5 +57,6 @@
     <visual><geometry><box size="0.1 ${base_y} 0.5"/></geometry>
       <material name="chair"/></visual>
-    <collision><geometry><box size="0.1 ${base_y} 0.5"/></geometry></collision>
+    <!-- Visual task geometry only: the execution chassis collision is the
+         base box and drive/support wheels below. -->
   </link>
   <joint name="seat_joint" type="fixed">
@@ -64,6 +67,7 @@
   <xacro:macro name="wheel" params="name y">
     <link name="${name}">
-      <inertial><mass value="2"/>
-        <inertia ixx="0.01" ixy="0" ixz="0" iyy="0.01" iyz="0" izz="0.02"/></inertial>
+      <inertial><mass value="1.5"/>
+        <!-- Cylinder axis is link y after the visual/collision rotation. -->
+        <inertia ixx="0.00875" ixy="0" ixz="0" iyy="0.03375" iyz="0" izz="0.00875"/></inertial>
       <visual>
         <origin rpy="1.5708 0 0"/>
@@ -91,5 +95,6 @@
   <xacro:wheel name="left_wheel" y="${sep/2}"/>
   <xacro:wheel name="right_wheel" y="${-sep/2}"/>
-  <!-- passive front caster (sphere) -->
+  <!-- Symmetric, friction-free support balls keep the simplified carrier
+       level without adding lateral rolling constraints. -->
   <link name="caster">
     <inertial><mass value="0.5"/>
@@ -104,5 +109,18 @@
     <origin xyz="${base_x/2 - 0.1} 0 ${-base_z/2 - wheel_r + 0.06}"/>
   </joint>
+  <link name="rear_caster">
+    <inertial><mass value="0.5"/>
+      <inertia ixx="0.001" ixy="0" ixz="0" iyy="0.001" iyz="0" izz="0.001"/></inertial>
+    <visual><geometry><sphere radius="0.06"/></geometry><material name="dark"/></visual>
+    <collision><geometry><sphere radius="0.06"/></geometry>
+      <surface><friction><ode><mu>0.0</mu><mu2>0.0</mu2></ode></friction></surface></collision>
+  </link>
+  <joint name="rear_caster_joint" type="fixed">
+    <parent link="base_link"/>
+    <child link="rear_caster"/>
+    <origin xyz="${-base_x/2 + 0.1} 0 ${-base_z/2 - wheel_r + 0.06}"/>
+  </joint>
   <gazebo reference="caster"><mu1>0.0</mu1><mu2>0.0</mu2></gazebo>
+  <gazebo reference="rear_caster"><mu1>0.0</mu1><mu2>0.0</mu2></gazebo>
   <gazebo reference="left_wheel">
     <mu1>$(arg wheel_mu)</mu1><mu2>$(arg wheel_mu)</mu2>
